File: MIST.kicad_sch (KiCad schematic)
At the start: 0 parts

Commit message: did some stuff
Parts:
- added D1: LED, LED_SMD:LED-APA102-2020, symbol Device:LED
- added R1: 220, Resistor_SMD:R_0201_0603Metric, symbol Device:R
Connections:
- new net +5V: R1.2
- new net GND: D1.1 (K)
- new net LED_Anode: D1.2 (A), R1.1
